File: projects/PCB Senior Design/Main.sch (EAGLE design)
At the start: 64 parts, among them J9 NANO_SIM, Q2 8MHz, Q3 2.5A/30V/105mΩ, U1 UBLOX_SAM_M8Q-0-10, U2 32KB NRF51822, U4 TCA9406DCU, U5 MCP73831, U6 SARA-R410M-2B, U7 TXB0104, U9 AP7361C-33FGE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

Commit message: Incorporated ESP32
Parts:
- removed C29, C30: 22p, SmartPrj:C-EU0603-RND
- removed C31: 100n, SmartPrj:C-EU0603-RND
- removed ICSP: 3x2 M, SmartPrj:PINHD-2X3
- removed Q2: 8MHz, special:XTAL
- removed R6: 10k, SparkFun-Resistors:10KOHM-0603-1/10W-1%
- removed RESET: TS42031-160R-TR-7260, SmartPrj:TS42
- removed RN1: 10K, resistor-dil:4R-NCAY16
- removed ZU4: ATMEGA328P-PU, SmartPrj:ATMEGA328P-PU
- added R8, R9: 220, rcl:R-US_R1206
- added U$4: ESP32-DEV-BOARD, SeniorDesign:ESP32-DEV-BOARD
- R7: value 1M -> 220; device SmartPrj:R-EU_R0603 -> rcl:R-US_R1206
Connections:
- removed net N$12: R6.2, U$1.O, U$1.S, U9.EN
- removed net RESET1: ICSP.5, RESET.3, RESET.4, RN1D.1, ZU4.RESET
- removed net XTAL1: C30.1, Q2.1, R7.1, ZU4.XTAL1
- removed net XTAL2: C29.1, Q2.2, R7.2, ZU4.XTAL2
- new net LED_B: R9.1, U$4.D27
- new net LED_G: R8.1, U$4.D26
- new net LED_R: R7.1, U$4.D25
- new net PWR-MODE1: U$1.O, U$4.D35
- new net PWR-MODE2: U$1.S, U$4.D14
- net 3.3V: now also U$3.P$2, U$4.3V3; no longer C31.2, ICSP.2, RN1D.2, U$3.P$1, ZU4.AVCC, ZU4.VCC
- net CS-BT: now also U$4.D2; no longer ZU4.(SS)PB2
- net GND: now also U$1.P, U$3.P$1, U$4.GND@1, U$4.GND@2; no longer C29.2, C30.2, C31.1, ICSP.6, R6.1, RESET.1, RESET.2, U$3.P$2, ZU4.AGND, ZU4.GND
- net IRQ-BT: now also U$4.D12; no longer ZU4.(AIN1)PD7
- net MISO: now also U$4.D19; no longer ICSP.1, ZU4.(MISO)PB4
- net MOSI: now also U$4.D23; no longer ICSP.4, ZU4.(MOSI)PB3
- net N$3: now also R7.2; no longer ZU4.(INT0)PD2
- net N$4: now also R8.2; no longer ZU4.(TXD)PD1
- net N$5: now also R9.2; no longer ZU4.(RXD)PD0
- net PING-POT: now also U$4.D34; no longer ZU4.(ADC0)PC0)
- net PWR-CELL: now also U$4.D32; no longer ZU4.(T1)PD5
- net RST-BT: now also U$4.D13; no longer ZU4.(T0)PD4
- net RST-CELL: now also U$4.D33; no longer ZU4.(AIN0)PD6
- net RX-ARD: now also U$4.RX0; no longer ZU4.(ICP)PB0
- net SCK: now also U$4.D18; no longer ICSP.3, ZU4.(SCK)PB5
- net TX-ARD: now also U$4.TX0; no longer ZU4.(OC1)PB1
- net VIN: now also U9.EN; no longer U$1.P
Other:
- note added: "Central MCU - ESP32"
- note removed: "Central MCU - ATMega328P"
